Commit message: add robot model

File: Assets/URDF/gopher_description/gopher.urdf (robot description, URDF)
Before this commit: robot gopher, 94 links, 93 joints
Links:
- removed link gopher/base_camera_optical_frame
- removed link gopher/left_arm_cam_color_frame
- removed link gopher/left_arm_cam_color_optical_frame
- removed link gopher/left_arm_cam_depth_frame
- removed link gopher/left_arm_cam_depth_optical_frame
- removed link gopher/left_arm_cam_left_ir_frame
- removed link gopher/left_arm_cam_left_ir_optical_frame
- removed link gopher/left_arm_cam_right_ir_frame
- removed link gopher/left_arm_cam_right_ir_optical_frame
- removed link gopher/left_arm_camera_color_frame
- removed link gopher/left_arm_camera_depth_frame
- removed link gopher/main_cam_color_frame
- removed link gopher/main_cam_color_optical_frame
- removed link gopher/main_cam_depth_frame
- removed link gopher/main_cam_depth_optical_frame
- removed link gopher/main_cam_left_ir_frame
- removed link gopher/main_cam_left_ir_optical_frame
- removed link gopher/main_cam_right_ir_frame
- removed link gopher/main_cam_right_ir_optical_frame
- removed link gopher/right_arm_cam_color_frame
- removed link gopher/right_arm_cam_color_optical_frame
- removed link gopher/right_arm_cam_depth_frame
- removed link gopher/right_arm_cam_depth_optical_frame
- removed link gopher/right_arm_cam_left_ir_frame
- removed link gopher/right_arm_cam_left_ir_optical_frame
- removed link gopher/right_arm_cam_right_ir_frame
- removed link gopher/right_arm_cam_right_ir_optical_frame
- removed link gopher/right_arm_camera_color_frame
- removed link gopher/right_arm_camera_depth_frame
Joints:
- removed joint gopher/base_camera_optical_joint
- removed joint gopher/left_arm_cam_color_joint
- removed joint gopher/left_arm_cam_color_optical_joint
- removed joint gopher/left_arm_cam_depth_joint
- removed joint gopher/left_arm_cam_depth_optical_joint
- removed joint gopher/left_arm_cam_left_ir_joint
- removed joint gopher/left_arm_cam_left_ir_optical_joint
- removed joint gopher/left_arm_cam_right_ir_joint
- removed joint gopher/left_arm_cam_right_ir_optical_joint
- removed joint gopher/left_arm_color_module
- removed joint gopher/left_arm_depth_module
- removed joint gopher/main_cam_color_joint
- removed joint gopher/main_cam_color_optical_joint
- removed joint gopher/main_cam_depth_joint
- removed joint gopher/main_cam_depth_optical_joint
- removed joint gopher/main_cam_left_ir_joint
- removed joint gopher/main_cam_left_ir_optical_joint
- removed joint gopher/main_cam_right_ir_joint
- removed joint gopher/main_cam_right_ir_optical_joint
- removed joint gopher/right_arm_cam_color_joint
- removed joint gopher/right_arm_cam_color_optical_joint
- removed joint gopher/right_arm_cam_depth_joint
- removed joint gopher/right_arm_cam_depth_optical_joint
- removed joint gopher/right_arm_cam_left_ir_joint
- removed joint gopher/right_arm_cam_left_ir_optical_joint
- removed joint gopher/right_arm_cam_right_ir_joint
- removed joint gopher/right_arm_cam_right_ir_optical_joint
- removed joint gopher/right_arm_color_module
- removed joint gopher/right_arm_depth_module
- joint gopher/left_shoulder_to_torso_joint: origin xyz=0 0 0.7 rpy=-1.57 0 0 -> xyz=0 0 0.7 rpy=-1.57 3.14 0

File: Assets/URDF/gopher_description/gopher_description/base/urdf/freight.urdf.xacro (robot description, xacro)
@@ -152,10 +152,4 @@
       <child link="${prefix}base_camera_link" />
     </joint>
-    <link name="${prefix}base_camera_optical_frame" />
-    <joint name="${prefix}base_camera_optical_joint" type="fixed">
-      <origin rpy="1.5707963267966 0 1.5707963267966" xyz="0 0 0" />
-      <parent link="${prefix}base_camera_link" />
-      <child link="${prefix}base_camera_optical_frame" />
-    </joint>
   </xacro:macro>
 </robot>

File: Assets/URDF/gopher_description/gopher_description/base/urdf/torso.urdf.xacro (robot description, xacro)
@@ -87,5 +87,5 @@
             <child link="${prefix}left_shoulder_link" />
             <parent link="${prefix}torso" />
-            <origin xyz="0 0 0.7" rpy="-1.57 0 0" />
+            <origin xyz="0 0 0.7" rpy="-1.57 3.14 0" />
             <axis xyz="0 0 1"/>
         </joint>

File: Assets/URDF/gopher_description/gopher_description/camera/urdf/_d435.urdf.xacro (robot description, xacro)
@@ -68,56 +68,4 @@
       </inertial>
     </link>
-    <!-- camera depth joints and links -->
-    <joint name="${prefix}depth_joint" type="fixed">
-      <origin xyz="0 0 0" rpy="0 0 0"/>
-      <parent link="${prefix}link"/>
-      <child link="${prefix}depth_frame" />
-    </joint>
-    <link name="${prefix}depth_frame"/>
-    <joint name="${prefix}depth_optical_joint" type="fixed">
-      <origin xyz="0 0 0" rpy="${-M_PI/2} 0 ${-M_PI/2}" />
-      <parent link="${prefix}depth_frame" />
-      <child link="${prefix}depth_optical_frame" />
-    </joint>
-    <link name="${prefix}depth_optical_frame"/>
-    <!-- camera left IR joints and links -->
-    <joint name="${prefix}left_ir_joint" type="fixed">
-      <origin xyz="0 ${d435_cam_depth_to_left_ir_offset} 0" rpy="0 0 0" />
-      <parent link="${prefix}depth_frame" />
-      <child link="${prefix}left_ir_frame" />
-    </joint>
-    <link name="${prefix}left_ir_frame"/>
-    <joint name="${prefix}left_ir_optical_joint" type="fixed">
-      <origin xyz="0 0 0" rpy="${-M_PI/2} 0 ${-M_PI/2}" />
-      <parent link="${prefix}left_ir_frame" />
-      <child link="${prefix}left_ir_optical_frame" />
-    </joint>
-    <link name="${prefix}left_ir_optical_frame"/>
-    <!-- camera right IR joints and links -->
-    <joint name="${prefix}right_ir_joint" type="fixed">
-      <origin xyz="0 ${d435_cam_depth_to_right_ir_offset} 0" rpy="0 0 0" />
-      <parent link="${prefix}depth_frame" />
-      <child link="${prefix}right_ir_frame" />
-    </joint>
-    <link name="${prefix}right_ir_frame"/>
-    <joint name="${prefix}right_ir_optical_joint" type="fixed">
-      <origin xyz="0 0 0" rpy="${-M_PI/2} 0 ${-M_PI/2}" />
-      <parent link="${prefix}right_ir_frame" />
-      <child link="${prefix}right_ir_optical_frame" />
-    </joint>
-    <link name="${prefix}right_ir_optical_frame"/>
-    <!-- camera color joints and links -->
-    <joint name="${prefix}color_joint" type="fixed">
-      <origin xyz="0 ${d435_cam_depth_to_color_offset} 0" rpy="0 0 0" />
-      <parent link="${prefix}depth_frame" />
-      <child link="${prefix}color_frame" />
-    </joint>
-    <link name="${prefix}color_frame"/>
-    <joint name="${prefix}color_optical_joint" type="fixed">
-      <origin xyz="0 0 0" rpy="${-M_PI/2} 0 ${-M_PI/2}" />
-      <parent link="${prefix}color_frame" />
-      <child link="${prefix}color_optical_frame" />
-    </joint>
-    <link name="${prefix}color_optical_frame"/>
   </xacro:macro>
 </robot>

File: Assets/URDF/gopher_description/kortex_description/arms/gen3/7dof/urdf/gen3_macro.xacro (robot description, xacro)
@@ -317,16 +317,4 @@
         <child  link="${prefix}camera_link" />
       </joint>
-      <link name="${prefix}camera_depth_frame" />
-      <joint name="${prefix}depth_module" type="fixed">
-        <origin xyz="0.0275 0.066 -0.00305" rpy="3.14159265358979 3.14159265358979 0" />
-        <parent link="${prefix}end_effector_link" />
-        <child  link="${prefix}camera_depth_frame" />
-      </joint>
-      <link name="${prefix}camera_color_frame" />
-      <joint name="${prefix}color_module" type="fixed">
-        <origin xyz="0 0.05639 -0.00305" rpy="3.14159265358979 3.14159265358979 0" />
-        <parent link="${prefix}end_effector_link" />
-        <child  link="${prefix}camera_color_frame" />
-      </joint>
     </xacro:if>
   </xacro:macro>
