Commit message: add robot prefab

File: Assets/URDF/gopher_description/fetch_description/urdf/freight.urdf.xacro (robot description, xacro)
@@ -49,5 +49,5 @@
     </link>
     <joint name="${prefix}r_wheel_joint" type="continuous">
-      <origin rpy="-6.123E-17 0 0" xyz="0.0012914 -0.18738 0.0602" /> <!-- r 0.0605 -->
+      <origin rpy="-6.123E-17 0 0" xyz="0.0012914 -0.18738 0.0605" />
       <parent link="${prefix}chassis_link" />
       <child link="${prefix}r_wheel_link" />
@@ -78,5 +78,5 @@
     </link>
     <joint name="${prefix}l_wheel_joint" type="continuous">
-      <origin rpy="-6.123E-17 0 0" xyz="0.0012914 0.18738 0.0602" /> <!-- r 0.0605 -->
+      <origin rpy="-6.123E-17 0 0" xyz="0.0012914 0.18738 0.0605" />
       <parent link="${prefix}chassis_link" />
       <child link="${prefix}l_wheel_link" />

File: Assets/URDF/gopher_description/realsense2_description/urdf/_d435.urdf_origin.xacro (robot description, xacro)
@@ -71,4 +71,36 @@
     </joint>
     <link name="${prefix}depth_frame"/>
+    <joint name="${prefix}depth_optical_joint" type="fixed">
+      <origin xyz="0 0 0" rpy="${-M_PI/2} 0 ${-M_PI/2}" />
+      <parent link="${prefix}depth_frame" />
+      <child link="${prefix}depth_optical_frame" />
+    </joint>
+    <link name="${prefix}depth_optical_frame"/>
+    <!-- camera left IR joints and links -->
+    <joint name="${prefix}left_ir_joint" type="fixed">
+      <origin xyz="0 ${d435_cam_depth_to_left_ir_offset} 0" rpy="0 0 0" />
+      <parent link="${prefix}depth_frame" />
+      <child link="${prefix}left_ir_frame" />
+    </joint>
+    <link name="${prefix}left_ir_frame"/>
+    <joint name="${prefix}left_ir_optical_joint" type="fixed">
+      <origin xyz="0 0 0" rpy="${-M_PI/2} 0 ${-M_PI/2}" />
+      <parent link="${prefix}left_ir_frame" />
+      <child link="${prefix}left_ir_optical_frame" />
+    </joint>
+    <link name="${prefix}left_ir_optical_frame"/>
+    <!-- camera right IR joints and links -->
+    <joint name="${prefix}right_ir_joint" type="fixed">
+      <origin xyz="0 ${d435_cam_depth_to_right_ir_offset} 0" rpy="0 0 0" />
+      <parent link="${prefix}depth_frame" />
+      <child link="${prefix}right_ir_frame" />
+    </joint>
+    <link name="${prefix}right_ir_frame"/>
+    <joint name="${prefix}right_ir_optical_joint" type="fixed">
+      <origin xyz="0 0 0" rpy="${-M_PI/2} 0 ${-M_PI/2}" />
+      <parent link="${prefix}right_ir_frame" />
+      <child link="${prefix}right_ir_optical_frame" />
+    </joint>
+    <link name="${prefix}right_ir_optical_frame"/>
     <!-- camera color joints and links -->
     <joint name="${prefix}color_joint" type="fixed">
@@ -78,4 +110,10 @@
     </joint>
     <link name="${prefix}color_frame"/>
+    <joint name="${prefix}color_optical_joint" type="fixed">
+      <origin xyz="0 0 0" rpy="${-M_PI/2} 0 ${-M_PI/2}" />
+      <parent link="${prefix}color_frame" />
+      <child link="${prefix}color_optical_frame" />
+    </joint>
+    <link name="${prefix}color_optical_frame"/>
   </xacro:macro>
 </robot>

File: Assets/URDF/kortex_description/arms/gen3/7dof/urdf/gen3_macro.xacro (robot description, xacro)
@@ -317,4 +317,15 @@
         <child  link="${prefix}camera_link" />
       </joint>
+      <link name="${prefix}camera_depth_frame" />
+      <joint name="${prefix}depth_module" type="fixed">
+        <origin xyz="0.0275 0.066 -0.00305" rpy="3.14159265358979 3.14159265358979 0" />
+        <parent link="${prefix}end_effector_link" />
+        <child  link="${prefix}camera_depth_frame" />
+      </joint>
+      <link name="${prefix}camera_color_frame" />
+      <joint name="${prefix}color_module" type="fixed">
+        <origin xyz="0 0.05639 -0.00305" rpy="3.14159265358979 3.14159265358979 0" />
+        <parent link="${prefix}end_effector_link" />
+        <child  link="${prefix}camera_color_frame" />
     </xacro:if>
   </xacro:macro>
