Commit message: load robot model

File: Assets/URDF/freight.urdf (robot description, URDF)
Before this commit: robot freight, 7 links, 6 joints
Links:
- removed link base_camera_link
- removed link base_camera_optical_frame
- removed link base_link
- removed link estop_link
- removed link l_wheel_link
- removed link laser_link
- removed link r_wheel_link
- added link freight/base_camera_link
- added link freight/base_camera_optical_frame
- added link freight/base_link
- added link freight/chassis_link, mass 70.1294; collision mesh filename=package://gopher_description/fetch_description/meshes/base_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; visual mesh filename=package://gopher_description/fetch_description/meshes/base_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
- added link freight/estop_link, mass 0.00196130439134723; collision mesh filename=package://gopher_description/fetch_description/meshes/estop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; visual mesh filename=package://gopher_description/fetch_description/meshes/estop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
- added link freight/l_wheel_link, mass 4.3542; collision mesh filename=package://gopher_description/fetch_description/meshes/l_whe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; visual mesh filename=package://gopher_description/fetch_description/meshes/l_whe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
- added link freight/laser_link, mass 0.00833634573995571; collision mesh filename=package://gopher_description/fetch_description/meshes/laser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; visual mesh filename=package://gopher_description/fetch_description/meshes/laser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
- added link freight/r_wheel_link, mass 4.3542; collision mesh filename=package://gopher_description/fetch_description/meshes/r_whe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; visual mesh filename=package://gopher_description/fetch_description/meshes/r_whe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
Joints:
- removed joint base_camera_joint
- removed joint base_camera_optical_joint
- removed joint estop_joint
- removed joint l_wheel_joint
- removed joint laser_joint
- removed joint r_wheel_joint
- added joint freight/base_camera_joint: type fixed, parent freight/chassis_link, child freight/base_camera_link, origin xyz=0.2645 0 0.198 rpy=0 -0.17453292519943 0
- added joint freight/base_camera_optical_joint: type fixed, parent freight/base_camera_link, child freight/base_camera_optical_frame, origin xyz=0 0 0 rpy=1.5707963267966 0 1.5707963267966
- added joint freight/base_joint: type fixed, parent freight/base_link, child freight/chassis_link
- added joint freight/estop_joint: type fixed, parent freight/chassis_link, child freight/estop_link, origin xyz=-0.12465 0.23892 0.31127 rpy=1.5708 0 0, axis 0 0 0
- added joint freight/l_wheel_joint: type continuous, parent freight/chassis_link, child freight/l_wheel_link, origin xyz=0.0012914 0.18738 0.0602 rpy=-6.123E-17 0 0, axis 0 1 0, limit effort=8.85 velocity=34.8
- added joint freight/laser_joint: type fixed, parent freight/chassis_link, child freight/laser_link, origin xyz=0.235 0 0.2878 rpy=3.14159265359 0 0, axis 0 0 0
- added joint freight/r_wheel_joint: type continuous, parent freight/chassis_link, child freight/r_wheel_link, origin xyz=0.0012914 -0.18738 0.0602 rpy=-6.123E-17 0 0, axis 0 1 0, limit effort=8.85 velocity=34.8

Commit message: fix robot urdf

File: Assets/URDF/freight.urdf (robot description, URDF)
Before this commit: robot gopher, 8 links, 7 joints
Links:
- link freight/base_camera_link: mass None -> 0.001
- link freight/base_camera_optical_frame: mass None -> 0.001
Joints:
- joint freight/l_wheel_joint: origin xyz=0.0012914 0.18738 0.0602 rpy=-6.123E-17 0 0 -> xyz=0.0012914 0.18738 0.0605 rpy=-6.123E-17 0 0
- joint freight/r_wheel_joint: origin xyz=0.0012914 -0.18738 0.0602 rpy=-6.123E-17 0 0 -> xyz=0.0012914 -0.18738 0.0605 rpy=-6.123E-17 0 0

File: Assets/URDF/gopher.urdf (robot description, URDF)
Before this commit: robot Gopher, 64 links, 63 joints
Links:
- link gopher/base_camera_link: mass None -> 0.001
- link gopher/base_camera_optical_frame: mass None -> 0.001
- link gopher/left_arm_camera_color_frame: mass None -> 0.001
- link gopher/left_arm_camera_depth_frame: mass None -> 0.001
- link gopher/left_arm_camera_link: mass None -> 0.001
- link gopher/left_arm_end_effector_link: mass None -> 0.001
- link gopher/left_arm_left_inner_finger_pad: mass None -> 0.001
- link gopher/left_arm_right_inner_finger_pad: mass None -> 0.001
- link gopher/left_arm_tool_frame: mass None -> 0.001
- link gopher/main_cam_bottom_screw_frame: mass None -> 0.001
- link gopher/main_cam_color_frame: mass None -> 0.001
- link gopher/main_cam_depth_frame: mass None -> 0.001
- link gopher/right_arm_camera_color_frame: mass None -> 0.001
- link gopher/right_arm_camera_depth_frame: mass None -> 0.001
- link gopher/right_arm_camera_link: mass None -> 0.001
- link gopher/right_arm_end_effector_link: mass None -> 0.001
- link gopher/right_arm_left_inner_finger_pad: mass None -> 0.001
- link gopher/right_arm_right_inner_finger_pad: mass None -> 0.001
- link gopher/right_arm_tool_frame: mass None -> 0.001
Joints:
- joint gopher/l_wheel_joint: origin xyz=0.0012914 0.18738 0.0602 rpy=-6.123E-17 0 0 -> xyz=0.0012914 0.18738 0.0605 rpy=-6.123E-17 0 0
- joint gopher/r_wheel_joint: origin xyz=0.0012914 -0.18738 0.0602 rpy=-6.123E-17 0 0 -> xyz=0.0012914 -0.18738 0.0605 rpy=-6.123E-17 0 0

File: Assets/URDF/gopher_description/fetch_description/urdf/freight.urdf.xacro (robot description, xacro)
@@ -140,5 +140,11 @@
       <axis xyz="0 0 0" />
     </joint>
-    <link name="${prefix}base_camera_link" />
+    <link name="${prefix}base_camera_link">
+      <inertial>
+        <origin xyz="0 0 0" rpy="0 0 0" />
+        <mass value="0.001" />
+        <inertia ixx="1E-5" ixy="0" ixz="0" iyy="1E-5" iyz="-0" izz="1E-5" />
+      </inertial>
+    </link>
     <joint name="${prefix}base_camera_joint" type="fixed">
       <origin rpy="0 -0.17453292519943 0" xyz="0.2645 0 0.198" />
@@ -146,5 +152,11 @@
       <child link="${prefix}base_camera_link" />
     </joint>
-    <link name="${prefix}base_camera_optical_frame" />
+    <link name="${prefix}base_camera_optical_frame">
+      <inertial>
+        <origin xyz="0 0 0" rpy="0 0 0" />
+        <mass value="0.001" />
+        <inertia ixx="1E-5" ixy="0" ixz="0" iyy="1E-5" iyz="-0" izz="1E-5" />
+      </inertial>
+    </link>
     <joint name="${prefix}base_camera_optical_joint" type="fixed">
       <origin rpy="1.5707963267966 0 1.5707963267966" xyz="0 0 0" />

File: Assets/URDF/gopher_description/realsense2_description/urdf/_d435.urdf.xacro (robot description, xacro)
@@ -35,5 +35,11 @@
       <child link="${prefix}bottom_screw_frame" />
     </joint>
-    <link name="${prefix}bottom_screw_frame"/>
+    <link name="${prefix}bottom_screw_frame">
+      <inertial>
+        <origin xyz="0 0 0" rpy="0 0 0" />
+        <mass value="0.001" />
+        <inertia ixx="1E-5" ixy="0" ixz="0" iyy="1E-5" iyz="-0" izz="1E-5" />
+      </inertial>
+    </link>
     <joint name="${prefix}link_joint" type="fixed">
       <origin xyz="0 ${d435_cam_depth_py} ${d435_cam_depth_pz}" rpy="0 0 0"/>
@@ -70,5 +76,11 @@
       <child link="${prefix}depth_frame" />
     </joint>
-    <link name="${prefix}depth_frame"/>
+    <link name="${prefix}depth_frame">
+      <inertial>
+        <origin xyz="0 0 0" rpy="0 0 0" />
+        <mass value="0.001" />
+        <inertia ixx="1E-5" ixy="0" ixz="0" iyy="1E-5" iyz="-0" izz="1E-5" />
+      </inertial>
+    </link>
     <!-- camera color joints and links -->
     <joint name="${prefix}color_joint" type="fixed">
@@ -77,5 +89,11 @@
       <child link="${prefix}color_frame" />
     </joint>
-    <link name="${prefix}color_frame"/>
+    <link name="${prefix}color_frame">
+      <inertial>
+        <origin xyz="0 0 0" rpy="0 0 0" />
+        <mass value="0.001" />
+        <inertia ixx="1E-5" ixy="0" ixz="0" iyy="1E-5" iyz="-0" izz="1E-5" />
+      </inertial>
+    </link>
   </xacro:macro>
 </robot>

File: Assets/URDF/kortex_description/arms/gen3/7dof/urdf/gen3_macro.xacro (robot description, xacro)
@@ -298,5 +298,11 @@
         velocity="1.2218" />
     </joint>
-    <link name="${prefix}end_effector_link" />
+    <link name="${prefix}end_effector_link">
+      <inertial>
+        <origin xyz="0 0 0" rpy="0 0 0" />
+        <mass value="0.001" />
+        <inertia ixx="1E-5" ixy="0" ixz="0" iyy="1E-5" iyz="-0" izz="1E-5" />
+      </inertial>
+    </link>
     <joint
       name="${prefix}end_effector"
@@ -311,5 +317,11 @@
     </joint>
     <xacro:if value="${vision}">
-      <link name="${prefix}camera_link" />
+      <link name="${prefix}camera_link">
+        <inertial>
+          <origin xyz="0 0 0" rpy="0 0 0" />
+          <mass value="0.001" />
+          <inertia ixx="1E-5" ixy="0" ixz="0" iyy="1E-5" iyz="-0" izz="1E-5" />
+        </inertial>
+      </link>
       <joint name="${prefix}camera_module" type="fixed">
         <origin xyz="0 0.05639 -0.00305" rpy="3.14159265358979 3.14159265358979 0" />
@@ -317,5 +329,11 @@
         <child  link="${prefix}camera_link" />
       </joint>
-      <link name="${prefix}camera_depth_frame" />
+      <link name="${prefix}camera_depth_frame">
+        <inertial>
+          <origin xyz="0 0 0" rpy="0 0 0" />
+          <mass value="0.001" />
+          <inertia ixx="1E-5" ixy="0" ixz="0" iyy="1E-5" iyz="-0" izz="1E-5" />
+        </inertial>
+      </link>
       <joint name="${prefix}depth_module" type="fixed">
         <origin xyz="0.0275 0.066 -0.00305" rpy="3.14159265358979 3.14159265358979 0" />
@@ -323,9 +341,16 @@
         <child  link="${prefix}camera_depth_frame" />
       </joint>
-      <link name="${prefix}camera_color_frame" />
+      <link name="${prefix}camera_color_frame">
+        <inertial>
+          <origin xyz="0 0 0" rpy="0 0 0" />
+          <mass value="0.001" />
+          <inertia ixx="1E-5" ixy="0" ixz="0" iyy="1E-5" iyz="-0" izz="1E-5" />
+        </inertial>
+      </link>
       <joint name="${prefix}color_module" type="fixed">
         <origin xyz="0 0.05639 -0.00305" rpy="3.14159265358979 3.14159265358979 0" />
         <parent link="${prefix}end_effector_link" />
         <child  link="${prefix}camera_color_frame" />
+      </joint>
     </xacro:if>
   </xacro:macro>

File: Assets/URDF/kortex_description/grippers/robotiq_2f_85/urdf/robotiq_arg2f_85_model_macro.xacro (robot description, xacro)
@@ -102,4 +102,9 @@
   <xacro:macro name="inner_finger_pad" params="prefix fingerprefix">
     <link name="${prefix}${fingerprefix}_inner_finger_pad">
+      <inertial>
+        <origin xyz="0 0 0" rpy="0 0 0" />
+        <mass value="0.001" />
+        <inertia ixx="1E-5" ixy="0" ixz="0" iyy="1E-5" iyz="-0" izz="1E-5" />
+      </inertial>
       <visual>
         <origin xyz="0 0 0" rpy="0 0 0" />
@@ -184,5 +189,11 @@
   <xacro:macro name="robotiq_arg2f_85" params="prefix parent">
     <!-- Tool frame used by the arm -->
-    <link name="${prefix}tool_frame"/>
+    <link name="${prefix}tool_frame">
+      <inertial>
+        <origin xyz="0 0 0" rpy="0 0 0" />
+        <mass value="0.001" />
+        <inertia ixx="1E-5" ixy="0" ixz="0" iyy="1E-5" iyz="-0" izz="1E-5" />
+      </inertial>
+    </link>
     <joint name="${prefix}tool_frame_joint" type="fixed">
         <origin xyz="0 0 0.120" rpy="0 0 0" />
